Commit message: add asus xtion sensor

File: nextbot_robot/robot_description/urdf/nextbot.xacro (robot description, xacro)
@@ -17,4 +17,28 @@
   <!-- Base footprint link-->
   <link name="base_footprint"/>
+      <joint name="asus_camera_joint" type="fixed">
+        <parent link="base_link"/>
+        <child link="asus_camera_link"/>
+        <origin xyz="0 0 0.7" rpy="0 0 0"/>
+      </joint>
+      <link name="asus_camera_link">
+        <inertial>
+          <mass value="0.200" />
+          <origin xyz="0 0 0" rpy="0 0 0" />
+          <inertia ixx="5.8083e-4" ixy="0" ixz="0" iyy="3.0833e-5" iyz="0" izz="5.9083e-4" />
+        </inertial>
+        <visual>
+          <origin xyz="0 0 0" rpy="0 0 0" />
+          <geometry>
+            <mesh filename="package://nextbot_robot/robot_description/mesh/asus_camera_simple.dae"/>
+          </geometry>
+        </visual>
+        <collision>
+          <origin xyz="0 0 0" rpy="0 0 0" />
+          <geometry>
+            <mesh filename="package://nextbot_robot/robot_description/mesh/asus_camera_simple.dae"/>
+          </geometry>
+        </collision>
+      </link>
   <link name="xv11">
     <collision>
@@ -36,5 +60,5 @@
       <origin xyz="0 0 0.07" rpy="0 0 0"/>
       <mass value="0.1"/>
-      <inertia ixx="0.2" ixy="0" ixz="0" iyy="0.2" iyz="0" izz="0.3"/>
+      <inertia ixx="0" ixy="0" ixz="0" iyy="0" iyz="0" izz="0"/>
     </inertial>
   </link>
@@ -94,7 +118,7 @@
     </visual>
     <inertial>
-      <origin xyz="0 0 0.07" rpy="0 0 0"/>
-      <mass value="52"/>
-      <inertia ixx="0.248" ixy="0" ixz="0" iyy="0.748" iyz="0" izz="0.748"/>
+      <origin xyz="-0.01 0 0.07" rpy="0 0 0"/>
+      <mass value="10"/>
+      <inertia ixx="0.01" ixy="0" ixz="0" iyy="10" iyz="0" izz="0.01"/>
     </inertial>
   </link>

Commit message: add asus camera topic

File: nextbot_robot/robot_description/urdf/nextbot.xacro (robot description, xacro)
@@ -41,4 +41,53 @@
         </collision>
       </link>
+      <joint name="asus_camera_depth_joint" type="fixed">
+        <origin xyz="0.0 0.049 0.0" rpy="0 0 0" />
+        <parent link="asus_camera_link" />
+        <child link="asus_camera_depth_frame"/>
+      </joint>
+      <link name="asus_camera_depth_frame"/>
+      <joint name="asus_camera_depth_optical_joint" type="fixed">
+        <origin xyz="0 0 0" rpy="${-PI/2} 0.0 ${-PI/2}" />
+        <parent link="asus_camera_depth_frame" />
+        <child link="asus_camera_depth_optical_frame"/>
+      </joint>
+      <link name="asus_camera_depth_optical_frame"/>
+      <joint name="asus_camera_rgb_joint" type="fixed">
+        <origin xyz="0.0 0.022 0.0" rpy="0 0 0" />
+        <parent link="asus_camera_link" />
+        <child link="asus_camera_rgb_frame"/>
+      </joint>
+      <link name="asus_camera_rgb_frame"/>
+      <joint name="asus_camera_rgb_optical_joint" type="fixed">
+        <origin xyz="0 0 0" rpy="${-PI/2} 0.0 ${-PI/2}" />
+        <parent link="asus_camera_rgb_frame" />
+        <child link="asus_camera_rgb_optical_frame"/>
+      </joint>
+      <link name="asus_camera_rgb_optical_frame"/>
+      <gazebo reference="asus_camera_depth_frame">
+        <sensor type="depth" name="asus_camera">
+          <update_rate>20</update_rate>
+          <camera>
+            <horizontal_fov>${62.8 * PI/180.0}</horizontal_fov>
+            <image>
+              <format>R8G8B8</format>
+              <width>640</width>
+              <height>480</height>
+            </image>
+            <clip>
+              <near>0.5</near>
+              <far>9</far>
+            </clip>
+          </camera>
+          <plugin name="asus_camera_camera_controller" filename="libgazebo_ros_openni_kinect.so">
+            <imageTopicName>asus_camera/rgb/image_raw</imageTopicName>
+            <cameraInfoTopicName>asus_camera/rgb/camera_info</cameraInfoTopicName>
+            <depthImageTopicName>asus_camera/depth/image_raw</depthImageTopicName>
+            <depthImageCameraInfoTopicName>asus_camera/depth/camera_info</depthImageCameraInfoTopicName>
+            <pointCloudTopicName>asus_camera/depth/points</pointCloudTopicName>
+            <frameName>asus_camera_depth_optical_frame</frameName>
+          </plugin>
+        </sensor>
+      </gazebo>
   <link name="xv11">
     <collision>
@@ -118,7 +167,7 @@
     </visual>
     <inertial>
-      <origin xyz="-0.01 0 0.07" rpy="0 0 0"/>
+      <origin xyz="-0.2 0 0.07" rpy="0 0 0"/>
       <mass value="10"/>
-      <inertia ixx="0.01" ixy="0" ixz="0" iyy="10" iyz="0" izz="0.01"/>
+      <inertia ixx="5" ixy="0" ixz="1" iyy="10" iyz="1" izz="1"/>
     </inertial>
   </link>

Commit message: Add table recognition

File: nextbot_robot/robot_description/urdf/nextbot.xacro (robot description, xacro)
@@ -20,5 +20,5 @@
         <parent link="base_link"/>
         <child link="asus_camera_link"/>
-        <origin xyz="0 0 0.7" rpy="0 0 0"/>
+        <origin xyz="0 0 1.2" rpy="0 0 0"/>
       </joint>
       <link name="asus_camera_link">
@@ -81,9 +81,4 @@
           </camera>
           <plugin name="asus_camera_controller" filename="libgazebo_ros_openni_kinect.so">
-            <imageTopicName>asus_camera/rgb/image_raw</imageTopicName>
-            <cameraInfoTopicName>asus_camera/rgb/camera_info</cameraInfoTopicName>
-            <depthImageTopicName>asus_camera/depth/image_raw</depthImageTopicName>
-            <depthImageCameraInfoTopicName>asus_camera/depth/camera_info</depthImageCameraInfoTopicName>
-            <pointCloudTopicName>asus_camera/depth/points</pointCloudTopicName>
             <frameName>asus_camera_depth_optical_frame</frameName>
           </plugin>

Commit message: add implement rtabmap

File: nextbot_robot/robot_description/urdf/nextbot.xacro (robot description, xacro)
@@ -17,10 +17,10 @@
   <!-- Base footprint link-->
   <link name="base_footprint"/>
-      <joint name="asus_camera_joint" type="fixed">
+      <joint name="camera_joint" type="fixed">
         <parent link="base_link"/>
-        <child link="asus_camera_link"/>
+        <child link="camera_link"/>
         <origin xyz="0 0 1.2" rpy="0 0 0"/>
       </joint>
-      <link name="asus_camera_link">
+      <link name="camera_link">
         <inertial>
           <mass value="0.200" />
@@ -41,30 +41,30 @@
         </collision>
       </link>
-      <joint name="asus_camera_depth_joint" type="fixed">
+      <joint name="camera_depth_joint" type="fixed">
         <origin xyz="0.0 0.049 0.0" rpy="0 0 0" />
-        <parent link="asus_camera_link" />
-        <child link="asus_camera_depth_frame"/>
+        <parent link="camera_link" />
+        <child link="camera_depth_frame"/>
       </joint>
-      <link name="asus_camera_depth_frame"/>
-      <joint name="asus_camera_depth_optical_joint" type="fixed">
+      <link name="camera_depth_frame"/>
+      <joint name="camera_depth_optical_joint" type="fixed">
         <origin xyz="0 0 0" rpy="${-PI/2} 0.0 ${-PI/2}" />
-        <parent link="asus_camera_depth_frame" />
-        <child link="asus_camera_depth_optical_frame"/>
+        <parent link="camera_depth_frame" />
+        <child link="camera_depth_optical_frame"/>
       </joint>
-      <link name="asus_camera_depth_optical_frame"/>
-      <joint name="asus_camera_rgb_joint" type="fixed">
+      <link name="camera_depth_optical_frame"/>
+      <joint name="camera_rgb_joint" type="fixed">
         <origin xyz="0.0 0.022 0.0" rpy="0 0 0" />
-        <parent link="asus_camera_link" />
-        <child link="asus_camera_rgb_frame"/>
+        <parent link="camera_link" />
+        <child link="camera_rgb_frame"/>
       </joint>
-      <link name="asus_camera_rgb_frame"/>
-      <joint name="asus_camera_rgb_optical_joint" type="fixed">
+      <link name="camera_rgb_frame"/>
+      <joint name="camera_rgb_optical_joint" type="fixed">
         <origin xyz="0 0 0" rpy="${-PI/2} 0.0 ${-PI/2}" />
-        <parent link="asus_camera_rgb_frame" />
-        <child link="asus_camera_rgb_optical_frame"/>
+        <parent link="camera_rgb_frame" />
+        <child link="camera_rgb_optical_frame"/>
       </joint>
-      <link name="asus_camera_rgb_optical_frame"/>
-      <gazebo reference="asus_camera_depth_frame">
-        <sensor type="depth" name="asus_camera">
+      <link name="camera_rgb_optical_frame"/>
+      <gazebo reference="camera_depth_frame">
+        <sensor type="depth" name="camera">
           <update_rate>20</update_rate>
           <camera>
@@ -80,6 +80,11 @@
             </clip>
           </camera>
-          <plugin name="asus_camera_controller" filename="libgazebo_ros_openni_kinect.so">
-            <frameName>asus_camera_depth_optical_frame</frameName>
+          <plugin name="camera_controller" filename="libgazebo_ros_openni_kinect.so">
+            <imageTopicName>camera/rgb/image_raw</imageTopicName>
+            <cameraInfoTopicName>camera/rgb/camera_info</cameraInfoTopicName>
+            <depthImageTopicName>camera/depth/image_raw</depthImageTopicName>
+            <depthImageCameraInfoTopicName>camera/depth/camera_info</depthImageCameraInfoTopicName>
+            <pointCloudTopicName>camera/depth/points</pointCloudTopicName>
+            <frameName>camera_depth_optical_frame</frameName>
           </plugin>
         </sensor>
